Commit message: working mapping

File: src/my_robot/urdf/project_robot.xacro (robot description, xacro)
@@ -124,5 +124,5 @@
         <dynamics damping="1.0" friction="1.0"/>
     </joint>
-    <!-- camera link and joint -->
+    <!-- rgb-d camera links and joints -->
     <link name="camera">
         <pose>0 0 0 0 0 0</pose>
@@ -150,4 +150,5 @@
         </collision>
     </link>
+    <link name="camera_optical"></link>
     <joint type="fixed" name="camera_joint">
         <origin xyz="0.225 0 0.1" rpy="0 0 0"/>
@@ -155,4 +156,9 @@
         <parent link="chassis"/>
         <axis xyz="0 1 0" rpy="0 0 0"/>
+    </joint>
+    <joint name="camera_optical_joint" type="fixed">
+        <origin xyz="0 0 0" rpy="-1.5707 0 -1.5707"/>
+        <parent link="camera"/>
+        <child link="camera_optical"/>
     </joint>
     <!-- hokuyo link and joint -->
